Commit message: update working version gazebo simulation for roboboat base on fishbot tutorial chapter 6. Able to use omni wheel controller to control model in Gazebo, next step is to migrate the capstone team's code to this repo

File: boat_ws/src/boat_description/urdf/boat/boat.urdf.xacro (robot description, xacro)
@@ -10,5 +10,7 @@
     <xacro:include filename="$(find boat_description)/urdf/boat/actuator/caster.urdf.xacro"/>
     <!-- plugin -->
-    <xacro:include filename="$(find boat_description)/urdf/boat/plugin/gazebo_control_plugin.xacro"/>
+    <!-- <xacro:include filename="$(find boat_description)/urdf/boat/plugin/gazebo_control_plugin.xacro"/> -->
+    <xacro:include filename="$(find boat_description)/urdf/boat/plugin/gazebo_sensor_plugin.xacro"/>
+    <xacro:include filename="$(find boat_description)/urdf/boat/boat.ros2_control.xacro"/>
     <!-- base macro -->
     <xacro:base_xacro length="0.12" radius="0.10"/>
@@ -22,4 +24,6 @@
     <xacro:caster_xacro caster_name="front_caster" xyz="0.08 0.0 -0.06"/>
     <xacro:caster_xacro caster_name="back_caster" xyz="-0.08 0.0 -0.06"/>
-    <xacro:gazebo_control_plugin/>
+    <!-- <xacro:gazebo_control_plugin/> -->
+    <xacro:gazebo_sensor_plugin/>
+    <xacro:boat_ros2_control/>
 </robot>

File: boat_ws/src/boat_description/urdf/boat/sensor/camera.urdf.xacro (robot description, xacro)
@@ -33,10 +33,16 @@
             <xacro:box_inertia m="0.1" w="0.02" h="0.10" d="0.02"/>
         </link>
+        <link name="camera_optical_link"></link>
         <!-- Joint to connect parts -->
         <!-- Type is either fixed or revolute-->
         <joint name="camera_joint" type="fixed">
-            <origin xyz="${xyz}" rpy="0.0 0.0 0.0"/>
             <parent link="base_link"/>
             <child link="camera_link"/>
+            <origin xyz="${xyz}" rpy="0.0 0.0 0.0"/>
+        </joint>
+        <joint name="camera_optical_joint" type="fixed">
+            <parent link="base_link"/>
+            <child link="camera_optical_link"/>
+            <origin xyz="0 0 0" rpy="${-pi/2} 0.0 ${-pi/2}"/>
         </joint>
     </xacro:macro>
